Commit message: urdf_updata script

File: LAFAN1_Visualize/robot_description/q1/q1.urdf (robot description, URDF)
Before this commit: robot q1, 20 links, 19 joints
Links:
- link left_ankle_link: mass 0.3360867  -> 0.4768037
- link left_elbow_link: mass 0.3412209 -> 0.3282012
- link left_hip_pitch_link: mass 1.8046 -> 1.871603
- link left_hip_roll_link: mass 2.1115 -> 2.1194499
- link left_hip_yaw_link: mass 2.3488936 -> 2.4878491
- link left_knee_link: mass 2.045647 -> 2.1687705
- link left_shoulder_pitch_link: mass 0.5404653 -> 0.5474344
- link left_shoulder_roll_link: mass 0.5428322 -> 0.5461248
- link left_shoulder_yaw_link: mass 0.6759657 -> 0.7134352
- link pelvis: mass 4.7536 -> 5.0175069
- link right_ankle_link: mass 0.3340051 -> 0.4768037
- link right_elbow_link: mass 0.3412209 -> 0.32819
- link right_hip_pitch_link: mass 1.7535642703233 -> 1.8719556
- link right_hip_roll_link: mass 2.1095097 -> 2.1194499
- link right_hip_yaw_link: mass 2.346563 -> 2.4854678
- link right_knee_link: mass 2.0286725 -> 2.1688182
- link right_shoulder_pitch_link: mass 0.5404653 -> 0.5474344
- link right_shoulder_roll_link: mass 0.5428322 -> 0.5461248
- link right_shoulder_yaw_link: mass 0.67597 -> 0.7134571
- link torso_link: mass 13.7367215 -> 13.5166565

File: LAFAN1_Visualize/robot_description/q2/q2.urdf (robot description, URDF)
Before this commit: robot q2, 22 links, 21 joints
Links:
- link left_ankle_pitch_link: mass 0.0329163 -> 0.0312897
- link left_ankle_roll_link: mass 0.314797 -> 0.445514
- link left_elbow_link: mass 0.3412209 -> 0.3282012
- link left_hip_pitch_link: mass 1.8046 -> 1.871603
- link left_hip_roll_link: mass 2.1115 -> 2.1194499
- link left_hip_yaw_link: mass 2.3488936 -> 2.4878491
- link left_knee_link: mass 2.045647 -> 2.1687705
- link left_shoulder_pitch_link: mass 0.5404653 -> 0.5474344
- link left_shoulder_roll_link: mass 0.5428322 -> 0.5461248
- link left_shoulder_yaw_link: mass 0.6759657 -> 0.7134352
- link pelvis: mass 4.7536 -> 5.0175069
- link right_ankle_pitch_link: mass 0.0329163 -> 0.0312897
- link right_ankle_roll_link: mass 0.314797 -> 0.445514
- link right_elbow_link: mass 0.3412209 -> 0.32819
- link right_hip_pitch_link: mass 1.7535642703233 -> 1.8719556
- link right_hip_roll_link: mass 2.1095097 -> 2.1194499
- link right_hip_yaw_link: mass 2.346563 -> 2.4854678
- link right_knee_link: mass 2.0286725 -> 2.1688182
- link right_shoulder_pitch_link: mass 0.5404653 -> 0.5474344
- link right_shoulder_roll_link: mass 0.5428322 -> 0.5461248
- link right_shoulder_yaw_link: mass 0.67597 -> 0.7134571
- link torso_link: mass 13.7367215 -> 13.5166565
